File: GarageDoor.brd (EAGLE design)
At the start: 56.8 x 63.5 mm, 39 parts, among them J1 DCJ0202, J2 RJ11-2L-B, J3 RJ11-2L-B

Commit message: Create PDF
Parts:
- J2, J3: device con-tycoelectronics:RJ11-NO_SHIELD -> KevinsLib:RJ11-NO_SHIELD
- moved Q6 21.1 mm to (23.5, 54.6), turned to 270 degrees
- moved R25 20.9 mm to (28.6, 57.1), turned to 0 degrees
- moved R22 18.7 mm to (42.5, 54.6), turned to 180 degrees
- moved R23 17.9 mm to (28.6, 54.0), turned to 0 degrees
- moved SV6 16.6 mm to (17.8, 61.0)
- moved R24 15.3 mm to (28.6, 51.4), turned to 0 degrees
- moved R19 14.9 mm to (42.5, 51.4), turned to 180 degrees
- moved SV4 13.5 mm to (47.0, 50.2), turned to 90 degrees
- moved R1 13.1 mm to (11.4, 55.2)
- moved R2 13.1 mm to (14.0, 55.2)
- moved R12 9.55 mm to (42.5, 46.4), turned to 180 degrees
- moved SV2 8.98 mm to (35.6, 61.0)
- moved R26 8.26 mm to (52.1, 29.2)
- moved R7 6.84 mm to (42.5, 58.4), turned to 180 degrees
- moved SV1 4.45 mm to (52.1, 38.7)
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Connections:
- removed net N$21: Q6.3, SV6.5
- new net A7: Q6.3, SC1.5, SV6.5
- net +5V: now also J1.1; no longer J1.3
- net GND: now also J1.3; no longer J1.1
Routing:
- net A7: track 0.00 -> 56.5 mm
- net GND: track 120.1 -> 66.3 mm, vias 4 -> 10
- net A6: track 19.2 -> 40.4 mm
- net A5: track 15.7 -> 32.9 mm
- net +5V: track 171.4 -> 156.3 mm
- net RX: track 43.8 -> 57.0 mm
- net TX: track 48.5 -> 60.3 mm
- net A4: track 12.1 -> 23.8 mm
- net A0: track 23.0 -> 34.7 mm
- net +3V3: track 155.6 -> 165.4 mm, vias 4 -> 6
- net N$21: track 8.35 -> 0.00 mm
- net N$2: track 10.9 -> 3.76 mm
- net N$4: track 10.6 -> 3.50 mm
- net N$3: track 9.52 -> 3.50 mm
- net A1: track 20.7 -> 15.0 mm
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- added copper zone on layer 1, net GND
Other:
- board size 56.8 x 63.5 mm -> 58.7 x 65.4 mm
