File: GarageDoor.sch (EAGLE design)
At the start: 39 parts, among them J1 DCJ0202, J2 RJ11-2L-B, J3 RJ11-2L-B

Commit message: Create PDF
Parts:
- J2, J3: device con-tycoelectronics:RJ11-2L-B -> KevinsLib:RJ11-2L-B
Connections:
- removed net N$21: Q6.D, SV6.5
- new net A7: Q6.D, SC1.A7, SV6.5
- net +5V: now also J1.1; no longer J1.3
- net GND: now also J1.3; no longer J1.1
Other:
- note added: "PCB Notes Center LED 90 Deg pin headers for camera and PIR Move those pin headers to top of the board, side by side Analog Read cad cell for light sensor"
- moved on the sheet: J1
Changed lines of the file:
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@@
 <layer number="223" name="223bmp" color="24" fill="1" visible="no" active="no"/>
 <layer number="224" name="224bmp" color="25" fill="1" visible="no" active="no"/>
+<layer number="231" name="Eagle3D_PG1" color="7" fill="1" visible="yes" active="yes"/>
+<layer number="232" name="Eagle3D_PG2" color="7" fill="1" visible="yes" active="yes"/>
+<layer number="233" name="Eagle3D_PG3" color="7" fill="1" visible="yes" active="yes"/>
 <layer number="248" name="Housing" color="7" fill="1" visible="yes" active="yes"/>
 <layer number="249" name="Edge" color="7" fill="1" visible="yes" active="yes"/>
@@
 <part name="P+1" library="supply1" deviceset="+5V" device=""/>
 <part name="+3V3" library="supply1" deviceset="+3V3" device=""/>
-<part name="J2" library="con-tycoelectronics" deviceset="RJ11" device="" technology="-2L-B"/>
-<part name="J3" library="con-tycoelectronics" deviceset="RJ11" device="" technology="-2L-B"/>
+<part name="J2" library="KevinsLib" deviceset="RJ11" device="" technology="-2L-B"/>
+<part name="J3" library="KevinsLib" deviceset="RJ11" device="" technology="-2L-B"/>
 <part name="+3V4" library="supply1" deviceset="+3V3" device=""/>
 <part name="SUPPLY4" library="supply2" deviceset="GND" device=""/>
@@
 Red LED Pin5
 Black LED Pin 6</text>
+<text x="132.08" y="12.7" size="1.778" layer="91">PCB Notes
+Center LED
+90 Deg pin headers for camera and PIR
+Move those pin headers to top of the board, side by side
+Analog Read cad cell for light sensor</text>
 </plain>
 <instances>
@@
 <instance part="SUPPLY10" gate="GND" x="139.7" y="48.26"/>
 <instance part="P+2" gate="1" x="-124.46" y="149.86"/>
-<instance part="J1" gate="G$1" x="-114.3" y="53.34"/>
+<instance part="J1" gate="G$1" x="-114.3" y="48.26"/>
 <instance part="SUPPLY2" gate="GND" x="-99.06" y="35.56"/>
 <instance part="R13" gate="G$1" x="119.38" y="66.04"/>
@@
 <pinref part="C3" gate="G$1" pin="-"/>
 <pinref part="SUPPLY2" gate="GND" pin="GND"/>
-<pinref part="J1" gate="G$1" pin="1"/>
-<wire x1="-106.68" y1="55.88" x2="-106.68" y2="63.5" width="0.1524" layer="91"/>
-<wire x1="-106.68" y1="63.5" x2="-121.92" y2="63.5" width="0.1524" layer="91"/>
-<wire x1="-121.92" y1="63.5" x2="-121.92" y2="43.18" width="0.1524" layer="91"/>
-<wire x1="-121.92" y1="43.18" x2="-99.06" y2="43.18" width="0.1524" layer="91"/>
-<wire x1="-99.06" y1="43.18" x2="-99.06" y2="38.1" width="0.1524" layer="91"/>
+<wire x1="-99.06" y1="43.18" x2="-99.06" y2="40.64" width="0.1524" layer="91"/>
+<pinref part="J1" gate="G$1" pin="3"/>
+<wire x1="-99.06" y1="40.64" x2="-99.06" y2="38.1" width="0.1524" layer="91"/>
+<wire x1="-106.68" y1="45.72" x2="-101.6" y2="45.72" width="0.1524" layer="91"/>
+<wire x1="-101.6" y1="45.72" x2="-101.6" y2="40.64" width="0.1524" layer="91"/>
+<wire x1="-101.6" y1="40.64" x2="-99.06" y2="40.64" width="0.1524" layer="91"/>
+<junction x="-99.06" y="40.64"/>
 </segment>
 <segment>
@@
 </segment>
 <segment>
-<pinref part="J1" gate="G$1" pin="3"/>
-<wire x1="-106.68" y1="50.8" x2="-99.06" y2="50.8" width="0.1524" layer="91"/>
 <wire x1="-99.06" y1="50.8" x2="-99.06" y2="55.88" width="0.1524" layer="91"/>
 <pinref part="C3" gate="G$1" pin="+"/>
+<pinref part="P+1" gate="1" pin="+5V"/>
+<pinref part="J1" gate="G$1" pin="1"/>
+<wire x1="-106.68" y1="50.8" x2="-99.06" y2="50.8" width="0.1524" layer="91"/>
 <junction x="-99.06" y="50.8"/>
-<pinref part="P+1" gate="1" pin="+5V"/>
 </segment>
 </net>
@@
 </segment>
 </net>
-<net name="N$21" class="0">
-<segment>
-<wire x1="53.34" y1="58.42" x2="48.26" y2="58.42" width="0.1524" layer="91"/>
-<wire x1="48.26" y1="58.42" x2="48.26" y2="40.64" width="0.1524" layer="91"/>
-<pinref part="Q6" gate="G$1" pin="D"/>
-<pinref part="SV6" gate="1" pin="5"/>
-</segment>
-</net>
 <net name="N$22" class="0">
 <segment>
@@
 </segment>
 </net>
+<net name="A7" class="0">
+<segment>
+<pinref part="SC1" gate="G$1" pin="A7"/>
+<wire x1="-121.92" y1="121.92" x2="-127" y2="121.92" width="0.1524" layer="91"/>
+<label x="-127" y="121.92" size="1.778" layer="95"/>
+</segment>
+<segment>
+<wire x1="53.34" y1="58.42" x2="48.26" y2="58.42" width="0.1524" layer="91"/>
+<wire x1="48.26" y1="58.42" x2="48.26" y2="43.18" width="0.1524" layer="91"/>
+<pinref part="Q6" gate="G$1" pin="D"/>
+<pinref part="SV6" gate="1" pin="5"/>
+<wire x1="48.26" y1="43.18" x2="48.26" y2="40.64" width="0.1524" layer="91"/>
+<wire x1="48.26" y1="43.18" x2="40.64" y2="43.18" width="0.1524" layer="91"/>
+<junction x="48.26" y="43.18"/>
+<label x="43.18" y="43.18" size="1.778" layer="95"/>
+</segment>
+</net>
